Commit message: new link and joint for updated camera

File: my_robot/urdf/my_robot.xacro (robot description, xacro)
@@ -33,4 +33,9 @@
     <axis xyz="0 1 0" rpy="0 0 0"/>
   </joint>
+  <joint name="camera_optical_joint" type="fixed">
+    <origin xyz="0 0 0" rpy="-1.5707 0 -1.5707"/>
+    <parent link="camera"/>
+    <child link="camera_link_optical"/>
+  </joint>
   <joint type="fixed" name="hokuyo_joint">
     <topicName>my_robot/laser/scan</topicName>
@@ -157,4 +162,5 @@
     </visual>
   </link>
+  <link name="camera_link_optical"></link>
   <link name='hokuyo'>
     <inertial>
